File: aquarium-lid.kicad_pcb (KiCad board)
At the start: 2 copper layers, 60 x 40 mm, 33 parts, among them J1 USB, J2 Fan1, J3 Fan2, J4 Temp Sensor, J5 USB_C_Receptacle_USB2.0_14P, J7 Extension, Q1 2N7002, Q2 2N7002, Q3 2N7002, SW1 Action 1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

Commit message: PCB updates
Routing:
- net +3V3: track 118.2 -> 116.9 mm
Other:
- board text added: "4.5-36V DC"
- board text added: "GND GND 3.3V 3.3V Vcc"
- board text added: "LEDs only run on 9.5-13.5V! Turn them off if input is not in that range."
- board text added: "SDA SCL IO2 IO3 IO5"
- board text removed: "3.3V"
- board text removed: "4.5-36V"
- board text removed: "GND"
- board text removed: "IO2"
- board text removed: "IO3"
- board text removed: "IO5"
- board text removed: "SCL"
- board text removed: "SDA"
- board text removed: "SRC"
Changed lines of the file:
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@@
 		(at 61 39 -90)
 		(property "Reference" "PS1"
-			(at -3 -6 180)
+			(at -3 -6 0)
 			(layer "F.SilkS")
 			(effects
@@
 		)
 		(embedded_fonts no)
+		(model "/home/mawoka/Documents/Kicad/easyeda2kicad/easyeda2kicad.3dshapes/PWRM-TH_3P-L11.5-W7.6-P2.54_R-78K3.3-0.5.wrl"
+			(offset
+				(xyz 0 0 10.2)
+			)
+			(scale
+				(xyz 1 1 1)
+			)
+			(rotate
+				(xyz -0 -0 -0)
+			)
+		)
 	)
 	(footprint "easyeda2kicad:LED-SMD_6P-L5.0-W5.0-P1.60-LS5.4-BR"
@@
 		(at 66.5875 57)
 		(property "Reference" "LED3"
-			(at -5.5875 1 0)
+			(at 5.4125 2 0)
 			(layer "F.SilkS")
 			(effects
@@
 			(at -3 0 0)
 			(layer "F.SilkS")
+			(hide yes)
 			(effects
 				(font
@@
 		(at 63.619 22)
 		(property "Reference" "U2"
-			(at 0 -5 0)
+			(at -1.619 4 0)
 			(layer "F.SilkS")
 			(effects
@@
 		(model "${EASYEDA2KICAD}/easyeda2kicad.3dshapes/IND-SMD_L7.8-W7.0-A.wrl"
 			(offset
-				(xyz 0 -0 -0)
+				(xyz 0 -0 3.5)
 			)
 			(scale
@@
 			)
 			(rotate
-				(xyz 0 0 0)
+				(xyz -0 -0 -0)
 			)
 		)
@@
 		)
 		(embedded_fonts no)
+		(model "/home/mawoka/Documents/Kicad/easyeda2kicad/easyeda2kicad.3dshapes/SW-SMD_4P-L6.0-W6.0-P4.50-LS11.0.wrl"
+			(offset
+				(xyz -3 0 2.3)
+			)
+			(scale
+				(xyz 1 1 1)
+			)
+			(rotate
+				(xyz -0 -0 -0)
+			)
+		)
 	)
 	(footprint "Capacitor_SMD:C_0805_2012Metric"
@@
 		(at 41 41 -90)
 		(property "Reference" "LS1"
-			(at -5 -7 180)
+			(at -5 -6 0)
 			(layer "F.SilkS")
 			(effects
@@
 		)
 		(fp_text user "+"
-			(at -5 -5 90)
+			(at -6 6 90)
 			(layer "F.SilkS")
 			(effects
@@
 		)
 		(fp_text user "-"
-			(at 7 3 90)
+			(at 4 6 90)
 			(layer "F.SilkS")
 			(effects
@@
 		)
 		(embedded_fonts no)
+		(model "/home/mawoka/Documents/Kicad/easyeda2kicad/easyeda2kicad.3dshapes/BUZ-TH_BD12.0-H6.0-P6.5.wrl"
+			(offset
+				(xyz 0 0 0)
+			)
+			(scale
+				(xyz 1 1 1)
+			)
+			(rotate
+				(xyz -0 -0 -90)
+			)
+		)
 	)
 	(footprint "Connector_JST:JST_PH_S3B-PH-SM4-TB_1x03-1MP_P2.00mm_Horizontal"
@@
 		(tags "connector JST PH horizontal")
 		(property "Reference" "J4"
-			(at 0 -5.8 90)
+			(at 2 -5.8 90)
 			(layer "F.SilkS")
 			(effects
@@
 		(embedded_fonts no)
 		(model "${KICAD9_3DMODEL_DIR}/Connector_JST.3dshapes/JST_PH_S3B-PH-SM4-TB_1x03-1MP_P2.00mm_Horizontal.wrl"
+			(hide yes)
 			(offset
 				(xyz 0 0 0)
@@
 			)
 		)
+		(model "/home/mawoka/Documents/Kicad/easyeda2kicad/easyeda2kicad.3dshapes/CONN-SMD_PH2.00-WS-3P.wrl"
+			(offset
+				(xyz 2 -2.9 0)
+			)
+			(scale
+				(xyz 1 1 1)
+			)
+			(rotate
+				(xyz -0 -0 -0)
+			)
+		)
 	)
 	(footprint "Resistor_SMD:R_0805_2012Metric"
@@
 			(at -3 0 0)
 			(layer "F.SilkS")
+			(hide yes)
 			(effects
 				(font
@@
 		(tags "ESP32-C3")
 		(property "Reference" "U1"
-			(at 0 -14.75 90)
+			(at -11 -2 90)
 			(layer "F.SilkS")
 			(effects
@@
 		(tags "connector JST XH horizontal")
 		(property "Reference" "J3"
-			(at -3.965 0.1 0)
+			(at 1.035 -2.9 0)
 			(layer "F.SilkS")
 			(effects
@@
 	)
 	(gr_rect
-		(start 42 35)
-		(end 50 43)
+		(start 47 37)
+		(end 55 45)
 		(stroke
 			(width 0.1)
@@
 		(layer "Edge.Cuts")
 	)
-	(gr_text "3.3V"
-		(at 74 54 90)
-		(layer "F.SilkS")
-		(effects
-			(font
-				(size 0.5 0.5)
-				(thickness 0.1)
-				(bold yes)
-			)
-			(justify left bottom)
-		)
-	)
-	(gr_text "IO3"
-		(at 74 56 90)
-		(layer "F.SilkS")
-		(effects
-			(font
-				(size 0.5 0.5)
-				(thickness 0.1)
-				(bold yes)
-			)
-			(justify left bottom)
-		)
-	)
-	(gr_text "SDA"
-		(at 71 56 90)
+	(gr_text "SDA\nSCL\nIO2\nIO3\nIO5"
+		(at 76 58 90)
 		(layer "F.SilkS")
 		(effects
 			(font
-				(size 0.5 0.5)
-				(thickness 0.1)
+				(size 0.7 0.7)
+				(thickness 0.15)
 				(bold yes)
 			)
@@
 	)
 	(gr_text "LEDs ON - LEDs OFF"
-		(at 55 55 0)
+		(at 53.346608 56 0)
 		(layer "F.SilkS")
 		(effects
 			(font
-				(size 0.5 0.5)
+				(size 0.6 0.6)
 				(thickness 0.1)
 			)
@@
 		)
 	)
-	(gr_text "IO5"
-		(at 75 56 90)
+	(gr_text "LEDs only run on 9.5-13.5V!\nTurn them off if input is not\nin that range."
+		(at 58.29375 59 0)
 		(layer "F.SilkS")
 		(effects
 			(font
-				(size 0.5 0.5)
-				(thickness 0.1)
+				(size 0.4 0.4)
+				(thickness 0.08)
 				(bold yes)
 			)
-			(justify left bottom)
-		)
-	)
-	(gr_text "3.3V"
-		(at 73 54 90)
-		(layer "F.SilkS")
-		(effects
-			(font
-				(size 0.5 0.5)
-				(thickness 0.1)
-				(bold yes)
-			)
-			(justify left bottom)
+			(justify bottom)
 		)
 	)
-	(gr_text "SCL"
-		(at 72 56 90)
+	(gr_text "4.5-36V DC"
+		(at 78 31 90)
 		(layer "F.SilkS")
 		(effects
 			(font
-				(size 0.5 0.5)
-				(thickness 0.1)
-				(bold yes)
-			)
-			(justify left bottom)
-		)
-	)
-	(gr_text "4.5-36V"
-		(at 78 29 90)
-		(layer "F.SilkS")
-		(effects
-			(font
-				(size 0.8 0.8)
-				(thickness 0.1)
-				(bold yes)
-			)
-			(justify left bottom)
-		)
-	)
-	(gr_text "GND"
-		(at 72 54 90)
-		(layer "F.SilkS")
-		(effects
-			(font
-				(size 0.5 0.5)
-				(thickness 0.1)
+				(size 1 1)
+				(thickness 0.2)
 				(bold yes)
 			)
@@
 		)
 	)
-	(gr_text "GND"
-		(at 71 54 90)
-		(layer "F.SilkS")
-		(effects
-			(font
-				(size 0.5 0.5)
-				(thickness 0.1)
-				(bold yes)
-			)
-			(justify left bottom)
-		)
-	)
-	(gr_text "SRC"
-		(at 75 54 90)
-		(layer "F.SilkS")
-		(effects
-			(font
-				(size 0.5 0.5)
-				(thickness 0.1)
-				(bold yes)
-			)
-			(justify left bottom)
-		)
-	)
-	(gr_text "IO2"
-		(at 73 56 90)
+	(gr_text "GND\nGND\n3.3V\n3.3V\nVcc"
+		(at 76 55 90)
 		(layer "F.SilkS")
 		(effects
 			(font
-				(size 0.5 0.5)
-				(thickness 0.1)
+				(size 0.7 0.7)
+				(thickness 0.15)
 				(bold yes)
 			)
@@
 	)
 	(gr_text "V1.1"
-		(at 53 23 180)
+		(at 78 58 0)
 		(layer "B.SilkS")
 		(effects
@@
 	)
 	(gr_text "Fancontroller by mawoka.eu"
-		(at 53 25 180)
+		(at 78 56 0)
 		(layer "B.SilkS")
 		(effects
@@
 	)
 	(segment
-		(start 41.076 49.924)
-		(end 42 49)
-		(width 0.4)
-		(layer "F.Cu")
-		(net 1)
-	)
-	(segment
 		(start 42.851 49.851)
 		(end 42 49)
@@
 	)
 	(segment
+		(start 50.33873 51)
+		(end 47.27421 47.93548)
+		(width 0.2)
+		(layer "B.Cu")
+		(net 38)
+	)
+	(segment
 		(start 79 46)
 		(end 79 44)
@@
 	)
 	(segment
-		(start 78 43)
-		(end 79 44)
+		(start 54 51)
+		(end 50.33873 51)
 		(width 0.2)
 		(layer "B.Cu")
@@
 	)
 	(segment
-		(start 60.782217 52.801)
-		(end 52.13973 52.801)
+		(start 55.801 52.801)
+		(end 54 51)
 		(width 0.2)
 		(layer "B.Cu")
@@
 	)
 	(segment
-		(start 33.85 35)
-		(end 30.1 31.25)
+		(start 78 43)
+		(end 79 44)
 		(width 0.2)
 		(layer "B.Cu")
@@
 	)
 	(segment
-		(start 52.13973 52.801)
-		(end 47.27421 47.93548)
+		(start 60.782217 52.801)
+		(end 55.801 52.801)
+		(width 0.2)
+		(layer "B.Cu")
+		(net 38)
+	)
+	(segment
+		(start 33.85 35)
+		(end 30.1 31.25)
 		(width 0.2)
 		(layer "B.Cu")
