File: aquarium-lid.kicad_pcb (KiCad board)
At the start: 2 copper layers, 60 x 40 mm, 29 parts, among them J2 Fan1, J3 Fan2, J4 Temp Sensor, J5 USB_C_Receptacle_USB2.0_14P, Q1 2N7002, Q2 2N7002, Q3 2N7002, SW1 Action 1, U1 ESP32-C3-WROOM-02

Commit message: Quick save
Parts:
- added J1: USB, Connector_PinHeader_2.54mm:PinHeader_1x03_P2.54mm_Vertical, F.Cu at (22.7, 28.3)
- added J7: Extension, Connector_PinHeader_2.54mm:PinHeader_2x05_P2.54mm_Vertical, F.Cu at (67.9, 50.3)
- added SW2: SS12D07VG4 087, easyeda2kicad:SW-TH_SS12D07VG4, F.Cu at (61.1, 51.0)
- moved R4 22.9 mm to (44.2, 33.6)
- moved R3 20.1 mm to (40.6, 33.6)
Connections:
- C1 pad 1: Net-(PS1-+VIN) -> GND
- DC1 pad 4: GND -> unconnected-(DC1-2-Pad4)
- J2 pad 1: +12V -> Net-(D4-A)
- J2 pad 2: Net-(D4-A) -> +12V
- J3 pad 1: +12V -> Net-(D3-A)
- J3 pad 2: Net-(D3-A) -> +12V
- LED1 pad 2: +12V -> Net-(LED1-VDD)
- LED2 pad 2: +12V -> Net-(LED1-VDD)
- LED3 pad 2: +12V -> Net-(LED1-VDD)
- U1 pad 11: unconnected-(U1-GPIO20/U0RXD-Pad11) -> /GPIO20
- U1 pad 12: unconnected-(U1-GPIO21/U0TXD-Pad12) -> /GPIO21
- U1 pad 15: unconnected-(U1-GPIO3/ADC1_CH3-Pad15) -> /GPIO3
- U1 pad 16: unconnected-(U1-GPIO2/ADC1_CH2-Pad16) -> /GPIO2
- U1 pad 4: unconnected-(U1-GPIO5/ADC2_CH0-Pad4) -> /GPIO5
Routing:
- net /GPIO2: track 0.00 -> 66.1 mm, vias 0 -> 2
- net /GPIO21: track 0.00 -> 61.6 mm, vias 0 -> 4
- net /GPIO3: track 0.00 -> 60.3 mm, vias 0 -> 3
- net /GPIO20: track 0.00 -> 54.0 mm, vias 0 -> 3
- net /GPIO5: track 0.00 -> 53.3 mm, vias 0 -> 5
- net Net-(LED1-VDD): track 0.00 -> 42.0 mm, vias 0 -> 2
- net GND: track 2.72 -> 39.4 mm, vias 25 -> 27
- net +12V: track 120.6 -> 84.4 mm, vias 4 -> 0
- net Net-(J5-CC2): track 5.98 -> 20.7 mm, vias 0 -> 2
- net /USB_D-: track 6.14 -> 20.7 mm
- net /USB_D+: track 7.61 -> 15.1 mm
- net Net-(PS1-+VIN): track 24.3 -> 16.9 mm
- net +3V3: track 74.0 -> 79.9 mm, vias 0 -> 2
- net Net-(D3-A): track 9.14 -> 13.2 mm, vias 0 -> 1
- net Net-(J5-CC1): track 9.55 -> 13.3 mm, vias 0 -> 2
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Other:
- board text added: "Fancontroller by mawoka.eu"
- board text added: "V1.1"

Commit message: New PCB
Parts:
- added U2: AHT20_C2757850, easyeda2kicad:SENSOR-SMD_L3.0-W3.0-P1.00-BR, F.Cu at (63.6, 22.0)
Connections:
- J7 pad 1: +3V3 -> /I2C_SDA
- J7 pad 10: /GPIO20 -> +12V
- J7 pad 2: +3V3 -> GND
- J7 pad 3: GND -> /I2C_SCL
- J7 pad 5: GND -> /GPIO2
- J7 pad 6: /GPIO5 -> +3V3
- J7 pad 8: /GPIO2 -> +3V3
- J7 pad 9: /GPIO21 -> /GPIO5
- R2 pad 1: GND -> +3V3
- U1 pad 11: /GPIO20 -> /I2C_SDA
- U1 pad 12: /GPIO21 -> /I2C_SCL
Routing:
- net /I2C_SCL: track 0.00 -> 103.3 mm, vias 0 -> 6
- net /I2C_SDA: track 0.00 -> 69.1 mm, vias 0 -> 5
- net /GPIO21: track 61.6 -> 0.00 mm, vias 4 -> 0
- net /GPIO20: track 54.0 -> 0.00 mm, vias 3 -> 0
- net +3V3: track 79.9 -> 118.2 mm, vias 2 -> 5
- net +12V: track 84.4 -> 102.0 mm
- net GND: track 39.4 -> 56.5 mm, vias 27 -> 31
- net /GPIO5: track 53.3 -> 62.9 mm
- net /GPIO2: track 66.1 -> 62.4 mm, vias 2 -> 4
Other:
- board text added: "3.3V"
- board text added: "4.5-36V"
- board text added: "GND"
- board text added: "GND D+ D-"
- board text added: "IO2"
- board text added: "IO3"
- board text added: "IO5"
- board text added: "LEDs ON - LEDs OFF"
- board text added: "SCL"
- board text added: "SDA"
- board text added: "SRC"

Commit message: Changes
Parts:
- moved J1 64.7 mm to (82.5, 53.1)
- moved J5 54.9 mm to (82.3, 40.0), turned to 90 degrees
- moved J4 47.8 mm to (29.5, 25.0), turned to 180 degrees
- moved R3 39.5 mm to (80.0, 31.5)
- moved R4 35.8 mm to (80.0, 33.5)
- moved U2 18.9 mm to (82.5, 23.0), turned to -90 degrees
Routing:
- net /USB_D+: track 15.1 -> 91.6 mm, vias 0 -> 1
- net /USB_D-: track 20.7 -> 87.7 mm, vias 0 -> 4
- net /I2C_SDA: track 69.1 -> 106.5 mm, vias 5 -> 7
- net /TEMP_DATA: track 45.8 -> 27.8 mm, vias 2 -> 4
- net Net-(J5-CC2): track 20.7 -> 6.22 mm, vias 2 -> 0
- net +3V3: track 118.2 -> 130.1 mm, vias 5 -> 10
- net GND: track 56.5 -> 51.2 mm, vias 31 -> 36
- net /I2C_SCL: track 103.3 -> 99.9 mm, vias 6 -> 4
- net Net-(J5-CC1): track 13.3 -> 16.4 mm
Other:
- board size 60 x 40 mm -> 66 x 40 mm
- board text added: "D+"
- board text added: "D-"
- board text removed: "GND D+ D-"
